File: micro_logger.sch (KiCad schematic (older format))
At the start: 25 parts, among them J4 Conn_01x02, J5 DM3AT-SF-PEJM5, SW2 SW_Push, U1 MIC5205-3.3, U2 TLV70218_SOT23-5, U4 ICM-20948, U5 PCA9306

Commit message: updated layout
Other:
- moved on the sheet: C1, C3, C4, D1, J5, R3, R4, SW2, U1
