File: hardware/_autosave-micro_logger.kicad_pcb (KiCad board)
At the start: 2 copper layers, 17.5 x 29.5 mm, 33 parts, among them J3 ISP, J4 Conn_01x02, J5 DM3AT-SF-PEJM5, SW2 SW_Push, U1 MIC5205-3.3, U2 TLV70218_SOT23-5, U3 ATMEGA328-AU, U4 ICM-20948, U5 PCA9306, Y1 Crystal_GND2

Commit message: added bom
Other:
- board text added: "+"
Changed lines of the file:
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@@
   (general
     (thickness 1.6)
-    (drawings 6)
+    (drawings 10)
     (tracks 415)
     (zones 0)
@@
     )
   )
+  (gr_text "+\n" (at 152.654 90.551) (layer F.SilkS)
+    (effects (font (size 0.5 0.5) (thickness 0.125)))
+  )
+  (gr_text "+\n" (at 154.305 90.551) (layer F.SilkS)
+    (effects (font (size 0.5 0.5) (thickness 0.125)))
+  )
+  (gr_text "+\n" (at 147.701 77.978) (layer F.SilkS)
+    (effects (font (size 0.5 0.5) (thickness 0.125)))
+  )
+  (gr_text "+\n" (at 141.478 74.676) (layer F.SilkS)
+    (effects (font (size 0.5 0.5) (thickness 0.125)))
+  )
   (gr_line (start 155.702 73.66) (end 138.176 73.66) (layer Edge.Cuts) (width 0.1))
