File: hardware/micro_logger.kicad_pcb (KiCad board)
At the start: 2 copper layers, 17.5 x 29.5 mm, 33 parts, among them J3 ISP, J4 Conn_01x02, J5 DM3AT-SF-PEJM5, SW2 SW_Push, U1 MIC5205-3.3, U2 TLV70218_SOT23-5, U3 ATMEGA328-AU, U4 ICM-20948, U5 PCA9306, Y1 Crystal_GND2

Commit message: updated symbols
Other:
- board text added: "+"
- board text added: "."
- board text added: "V1.1"
- board text removed: "V1"
Changed lines of the file:
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@@
-(kicad_pcb (version 20171130) (host pcbnew 5.0.1)
+(kicad_pcb (version 20171130) (host pcbnew 6.0.0-rc1-unknown-4ad37bc~66~ubuntu18.04.1)
   (general
     (thickness 1.6)
-    (drawings 6)
+    (drawings 12)
     (tracks 415)
     (zones 0)
@@
     (34 B.Paste user)
     (35 F.Paste user)
-    (36 B.SilkS user hide)
+    (36 B.SilkS user)
     (37 F.SilkS user)
     (38 B.Mask user hide)
@@
     (zone_45_only no)
     (trace_min 0.2)
-    (segment_width 0.2)
-    (edge_width 0.1)
     (via_size 0.8)
     (via_drill 0.4)
@@
     (uvia_min_size 0.2)
     (uvia_min_drill 0.1)
+    (edge_width 0.1)
+    (segment_width 0.2)
     (pcb_text_width 0.3)
     (pcb_text_size 1.5 1.5)
@@
       (effects (font (size 0.480833 0.480833) (thickness 0.05)))
     )
-    (fp_text value Crystal_GND2 (at 0.254 -6.096 270) (layer F.SilkS)
+    (fp_text value Crystal_GND2 (at 0.254 -6.096 270) (layer F.SilkS) hide
       (effects (font (size 0.481085 0.481085) (thickness 0.05)))
     )
@@
     (tags resistor)
     (attr smd)
-    (fp_text reference R9 (at 0 0.0762 90) (layer F.SilkS)
+    (fp_text reference R9 (at 0.03834 0.04064 180) (layer F.SilkS)
       (effects (font (size 0.5 0.5) (thickness 0.125)))
     )
@@
     (descr "Micro SD card holder with push-to-eject feature.")
     (attr smd)
-    (fp_text reference J5 (at -10.922 -2.46515 90) (layer B.SilkS) hide
-      (effects (font (size 1.0021 1.0021) (thickness 0.05)) (justify mirror))
+    (fp_text reference J5 (at 0.57404 -5.80064 180) (layer B.SilkS)
+      (effects (font (size 3 3) (thickness 0.05)) (justify mirror))
     )
     (fp_text value DM3AT-SF-PEJM5 (at 10.033 -2.331 90) (layer B.SilkS) hide
@@
     (descr "Through hole straight pin header, 2x03, 2.54mm pitch, double rows")
     (tags "Through hole pin header THT 2x03 2.54mm double row")
-    (fp_text reference J3 (at -0.05842 -0.11684) (layer F.SilkS)
+    (fp_text reference J3 (at 0.99822 -5.4864) (layer F.SilkS)
       (effects (font (size 1 1) (thickness 0.15)))
     )
@@
     )
   )
+  (gr_text + (at 152.6413 90.6145) (layer F.SilkS)
+    (effects (font (size 0.5 0.5) (thickness 0.125)))
+  )
+  (gr_text + (at 154.3431 90.5764) (layer F.SilkS)
+    (effects (font (size 0.5 0.5) (thickness 0.125)))
+  )
+  (gr_text + (at 147.701 77.6859) (layer F.SilkS)
+    (effects (font (size 0.5 0.5) (thickness 0.125)))
+  )
+  (gr_text + (at 141.6939 74.6633) (layer F.SilkS)
+    (effects (font (size 0.5 0.5) (thickness 0.125)))
+  )
+  (gr_text ".\n" (at 150.4569 90.3478) (layer F.SilkS)
+    (effects (font (size 1 1) (thickness 0.15)))
+  )
+  (gr_text ".\n" (at 142.8496 95.9231) (layer F.SilkS)
+    (effects (font (size 1 1) (thickness 0.15)))
+  )
   (gr_line (start 155.702 73.66) (end 138.176 73.66) (layer Edge.Cuts) (width 0.1))
   (gr_line (start 155.702 103.124) (end 155.702 73.66) (layer Edge.Cuts) (width 0.1))
   (gr_line (start 138.176 103.124) (end 155.702 103.124) (layer Edge.Cuts) (width 0.1))
   (gr_line (start 138.176 73.66) (end 138.176 103.124) (layer Edge.Cuts) (width 0.1))
-  (gr_text V1 (at 153.924 104.648) (layer F.SilkS)
+  (gr_text "V1.1\n" (at 153.99512 102.24516) (layer F.SilkS)
     (effects (font (size 0.5 0.5) (thickness 0.125)))
   )
