File: hardware/micro_logger.sch (KiCad schematic (older format))
At the start: 25 parts, among them J4 Conn_01x02, J5 DM3AT-SF-PEJM5, SW2 SW_Push, U1 MIC5205-3.3, U2 TLV70218_SOT23-5, U4 ICM-20948, U5 PCA9306

Commit message: merged in firmware
Parts:
- U2: symbol regul:TLV70218_SOT23-5 -> micro_logger-rescue:TLV70218_SOT23-5-regul
Changed lines of the file:
@@
 $EndComp
 $Comp
-L regul:TLV70218_SOT23-5 U2
+L micro_logger-rescue:TLV70218_SOT23-5-regul U2
 U 1 1 5BC82A48
 P 2700 2300

Commit message: updated schematic
Parts:
- added R?: 10k, Resistor_SMD:R_0805_2012Metric, symbol Device:R
- J4: value Conn_01x02 -> power
Connections:
- net Ardunio/D2: now also R?.2
- net GND: now also R?.1
Other:
- note added: "1.0\n"
- note added: "Micro Logger ICM-20498\n"
- note added: "Power Supply\n"
- moved on the sheet: C1, C11, C12, C13, C2, C3, C4, C5, C6, C7, D1, J4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
