File: hardware/Ardunio.sch (KiCad schematic (older format))
At the start: 10 parts, among them J3 ISP, U3 ATMEGA328-AU, Y1 Crystal_GND2

Commit message: updated schematic
Parts:
- JP1: value Jumper_NO_Small -> Reset_Jumper
- Y1: value Crystal_GND2 -> CSTCE8M00G55-R0
Other:
- note added: "Filter Capacitor"
- note added: "Programming Header\n"
- moved on the sheet: C10, C8, C9, D3, J3, JP1, R8, R9, U3, Y1
